File: mipi_spartan7/mipi_spartan7.kicad_pcb (KiCad board)
At the start: 4 copper layers, 30 x 45 mm, 130 parts, among them J1 SFW15R-1STE1LF, J2 DF40C-60DP-0.4V(51), J3 <DNP> PIN1X2, J4 0878325622, J5 <DNP> SSQ-106-02-F-D-RA, U1 XC7S6-2FTGB196C, U2 IS25LP016D-JULE-TR, U6 AP3401DNTR-G1, U7 AP3401DNTR-G1, U8 TPS22918DBV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

Commit message: 電源回路を昇圧DC-DCを使うものに変更
Parts:
- R25, R26: value 4.7k -> 2.2k
Connections:
- net /RPI_MIPI_CLK renamed /RPI_MIPI_GPIO1
- net /RPI_MIPI_GPIO renamed /RPI_MIPI_GPIO0
Other:
- board text added: "RTCL-S7-MIPI-V2"
- board text added: "©RTC-Lab"
- board text removed: "RTCL-MIPI-S7-V2"
- board text removed: "©Ryuz88"
