File: mipi_spartan7/mipi_spartan7.kicad_sch (KiCad schematic)
At the start: 126 parts, among them J1 SFW15R-1STE1LF, J2 DF40C-60DP-0.4V(51), J3 <DNP> PIN1X2, J4 0878325622, J5 <DNP> SSQ-106-02-F-D-RA, U1 XC7S6-2FTGB196C, U2 IS25LP016D-JULE-TR, U6 AP3401DNTR-G1, U7 AP3401DNTR-G1, U8 TPS22918DBV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

Commit message: 電源回路を昇圧DC-DCを使うものに変更
Parts:
- J1: footprint CON15_1X15_DRB_SFW_GLE -> mipi_spartan7:SFW15R-1STE1LF
- R25, R26: value 4.7k -> 2.2k
- U1: footprint FTGB196_XIL -> mipi_spartan7:FTGB196
- X1, X2: footprint Oscillator:Oscillator_SMD_SeikoEpson_SG8002LB-4Pin_5.0x3.2mm -> mipi_spartan7:SG-210STF
Connections:
- net RPI_MIPI_CLK renamed RPI_MIPI_GPIO1
- net RPI_MIPI_GPIO renamed RPI_MIPI_GPIO0
Changed lines of the file:
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@@
 		)
 	)
-	(label "RPI_MIPI_CLK"
+	(label "RPI_MIPI_GPIO1"
 		(at 173.99 199.39 0)
 		(effects
@@
 		)
 	)
-	(label "RPI_MIPI_GPIO"
+	(label "RPI_MIPI_GPIO0"
 		(at 173.99 204.47 0)
 		(effects
@@
 		)
 	)
-	(label "RPI_MIPI_CLK"
+	(label "RPI_MIPI_GPIO1"
 		(at 80.01 127 180)
 		(effects
@@
 		)
 	)
-	(label "RPI_MIPI_GPIO"
+	(label "RPI_MIPI_GPIO0"
 		(at 80.01 124.46 180)
 		(effects
@@
 			)
 		)
-		(property "Footprint" "Oscillator:Oscillator_SMD_SeikoEpson_SG8002LB-4Pin_5.0x3.2mm"
+		(property "Footprint" "mipi_spartan7:SG-210STF"
 			(at 360.68 316.23 0)
 			(effects
@@
 			)
 		)
-		(property "Value" "4.7k"
+		(property "Value" "2.2k"
 			(at 161.798 106.934 90)
 			(effects
@@
 			)
 		)
-		(property "Footprint" "FTGB196_XIL"
+		(property "Footprint" "mipi_spartan7:FTGB196"
 			(at 375.158 68.072 0)
 			(effects
@@
 			)
 		)
-		(property "Footprint" "CON15_1X15_DRB_SFW_GLE"
+		(property "Footprint" "mipi_spartan7:SFW15R-1STE1LF"
 			(at 29.464 85.852 0)
 			(effects
@@
 			)
 		)
-		(property "Footprint" "FTGB196_XIL"
+		(property "Footprint" "mipi_spartan7:FTGB196"
 			(at 212.598 68.072 0)
 			(effects
@@
 			)
 		)
-		(property "Footprint" "FTGB196_XIL"
+		(property "Footprint" "mipi_spartan7:FTGB196"
 			(at 211.328 233.172 0)
 			(effects
@@
 			)
 		)
-		(property "Value" "4.7k"
+		(property "Value" "2.2k"
 			(at 161.798 109.22 90)
 			(effects
@@
 			)
 		)
-		(property "Footprint" "Oscillator:Oscillator_SMD_SeikoEpson_SG8002LB-4Pin_5.0x3.2mm"
+		(property "Footprint" "mipi_spartan7:SG-210STF"
 			(at 360.68 275.59 0)
 			(effects
@@
 			)
 		)
-		(property "Footprint" "FTGB196_XIL"
+		(property "Footprint" "mipi_spartan7:FTGB196"
 			(at 511.048 65.532 0)
 			(effects

Commit message: update README
Parts:
- J4: JLC (none) -> C17275712
- L3, L4: JLC (none) -> C576403
- U1: JLC (none) -> C1521961
- U2: JLC (none) -> C2063555
- U6, U7: JLC (none) -> C507877
- U8: value TPS22918DBV -> TPS22918DBVR; JLC (none) -> C131941
- X1: JLC (none) -> C17669095
- X2: JLC (none) -> C17270014
Changed lines of the file:
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@@
 			)
 		)
+		(property "JLC" "C17275712"
+			(at 130.81 262.89 0)
+			(effects
+				(font
+					(size 1.27 1.27)
+				)
+				(hide yes)
+			)
+		)
 		(pin "11"
 		)
@@
 			)
 		)
+		(property "JLC" "C17270014"
+			(at 342.9 307.34 0)
+			(effects
+				(font
+					(size 1.27 1.27)
+				)
+				(hide yes)
+			)
+		)
 		(pin "4"
 		)
@@
 			)
 		)
+		(property "JLC" "C576403"
+			(at 494.03 279.4 90)
+			(effects
+				(font
+					(size 1.27 1.27)
+				)
+				(hide yes)
+			)
+		)
 		(pin "1"
 		)
@@
 			)
 		)
+		(property "JLC" "C1521961"
+			(at 387.35 85.09 0)
+			(effects
+				(font
+					(size 1.27 1.27)
+				)
+				(hide yes)
+			)
+		)
 		(pin "G8"
 		)
@@
 			)
 		)
+		(property "JLC" "C1521961"
+			(at 224.79 85.09 0)
+			(effects
+				(font
+					(size 1.27 1.27)
+				)
+				(hide yes)
+			)
+		)
 		(pin "G8"
 		)
@@
 			)
 		)
-		(property "Value" "TPS22918DBV"
+		(property "Value" "TPS22918DBVR"
 			(at 476.25 308.61 0)
 			(effects
@@
 			)
 		)
+		(property "JLC" " C131941"
+			(at 476.25 316.23 0)
+			(effects
+				(font
+					(size 1.27 1.27)
+				)
+				(hide yes)
+			)
+		)
 		(pin "4"
 		)
@@
 			)
 		)
+		(property "JLC" "C576403"
+			(at 494.03 248.92 90)
+			(effects
+				(font
+					(size 1.27 1.27)
+				)
+				(hide yes)
+			)
+		)
 		(pin "1"
 		)
@@
 			)
 		)
+		(property "JLC" "C1521961"
+			(at 223.52 250.19 0)
+			(effects
+				(font
+					(size 1.27 1.27)
+				)
+				(hide yes)
+			)
+		)
 		(pin "G8"
 		)
@@
 			)
 		)
+		(property "JLC" "C2063555"
+			(at 130.81 322.58 0)
+			(effects
+				(font
+					(size 1.27 1.27)
+				)
+				(hide yes)
+			)
+		)
 		(pin "5"
 		)
@@
 			)
 		)
+		(property "JLC" "C507877"
+			(at 476.25 283.21 0)
+			(effects
+				(font
+					(size 1.27 1.27)
+				)
+				(hide yes)
+			)
+		)
 		(pin "2"
 		)
@@
 			)
 		)
+		(property "JLC" "C507877"
+			(at 476.25 252.73 0)
+			(effects
+				(font
+					(size 1.27 1.27)
+				)
+				(hide yes)
+			)
+		)
 		(pin "2"
 		)
@@
 			)
 		)
+		(property "JLC" "C17669095"
+			(at 342.9 266.7 0)
+			(effects
+				(font
+					(size 1.27 1.27)
+				)
+				(hide yes)
+			)
+		)
 		(pin "4"
 		)
@@
 			(effects
 				(font
+					(size 1.27 1.27)
+				)
+				(hide yes)
+			)
+		)
+		(property "JLC" "C1521961"
+			(at 523.24 82.55 0)
+			(effects
+				(font
